File: pcb/kb.kicad_pcb (KiCad board)
At the start: 2 copper layers, 163.8 x 99.1 mm, 2 parts, among them SW1 SW_Push, U1 Pico

Commit message: Added Ergogen config + Fixes
What:

Why:

How:

Tags:
Other:
- net class Default removed
